Commit message: Officially done with MuJuCoo

File: mujoco_ws/mujoco_ros2_control_examples/panda_resources/panda_moveit_config/config/panda_arm_hand.srdf.xacro (robot description, xacro)
@@ -23,6 +23,6 @@
   </group_state>
   <group_state name="close" group="hand">
-    <joint name="panda_finger_joint1" value="0" />
-    <joint name="panda_finger_joint2" value="0" />
+    <joint name="panda_finger_joint1" value="0.014" />
+    <joint name="panda_finger_joint2" value="0.014" />
   </group_state>
   <!--END EFFECTOR: Purpose: Represent information about an end effector.-->

File: mujoco_ws/mujoco_ros2_control_examples/panda_resources/panda_moveit_config/config/panda_hand.ros2_control.xacro (robot description, xacro)
@@ -28,8 +28,8 @@
                 </xacro:unless>
                 <state_interface name="position">
-                  <param name="initial_value">0.0</param>
+                  <param name="initial_value">0.035</param>
                 </state_interface>
                 <state_interface name="velocity">
-                    <param name="initial_value">0.0</param>
+                    <param name="initial_value">0.035</param>
                 </state_interface>
             </joint>
@@ -48,8 +48,8 @@
                 </xacro:unless>
                 <state_interface name="position">
-                  <param name="initial_value">0.0</param>
+                  <param name="initial_value">0.035</param>
                 </state_interface>
                 <state_interface name="velocity">
-                    <param name="initial_value">0.0</param>
+                    <param name="initial_value">0.035</param>
                 </state_interface>
             </joint>
