Commit message: Added real shit

File: final_task/src/custom_arm_description/urdf/arm_urdf.xacro (robot description, xacro)
@@ -12,5 +12,5 @@
             <origin xyz="0.0 0.0 0.0" rpy="0.0 0.0 0.0" />
             <geometry>
-                <mesh filename="file://$(find arm_urdf)/meshes/base_link.stl" scale="0.001 0.001 0.001" />
+                <mesh filename="package://custom_arm_description/meshes/base_link.stl" scale="0.001 0.001 0.001" />
             </geometry>
         </visual>
@@ -18,5 +18,5 @@
             <origin xyz="0.0 0.0 0.0" rpy="0.0 0.0 0.0" />
             <geometry>
-                <mesh filename="file://$(find arm_urdf)/meshes/base_link.stl" scale="0.001 0.001 0.001" />
+                <mesh filename="package://custom_arm_description/meshes/base_link.stl" scale="0.001 0.001 0.001" />
             </geometry>
         </collision>
@@ -37,5 +37,5 @@
             <origin xyz="-0.03753819887451623 0.16137187769409533 0.0499999984935301" rpy="-1.5707963267948972 2.263292261842604e-15 -1.4329016358931765" />
             <geometry>
-                <mesh filename="file://$(find arm_urdf)/meshes/link1.stl" scale="0.001 0.001 0.001" />
+                <mesh filename="package://custom_arm_description/meshes/link1.stl" scale="0.001 0.001 0.001" />
             </geometry>
         </visual>
@@ -43,5 +43,5 @@
             <origin xyz="-0.03753819887451623 0.16137187769409533 0.0499999984935301" rpy="-1.5707963267948972 2.263292261842604e-15 -1.4329016358931765" />
             <geometry>
-                <mesh filename="file://$(find arm_urdf)/meshes/link1.stl" scale="0.001 0.001 0.001" />
+                <mesh filename="package://custom_arm_description/meshes/link1.stl" scale="0.001 0.001 0.001" />
             </geometry>
         </collision>
@@ -56,5 +56,5 @@
             <origin xyz="0.1659174891709117 -0.034739498800760875 0.250328893450339" rpy="0.13791264956862428 -0.016086890255214512 -0.002232659248270158" />
             <geometry>
-                <mesh filename="file://$(find arm_urdf)/meshes/link2.stl" scale="0.001 0.001 0.001" />
+                <mesh filename="package://custom_arm_description/meshes/link2.stl" scale="0.001 0.001 0.001" />
             </geometry>
         </visual>
@@ -62,5 +62,5 @@
             <origin xyz="0.1659174891709117 -0.034739498800760875 0.250328893450339" rpy="0.13791264956862428 -0.016086890255214512 -0.002232659248270158" />
             <geometry>
-                <mesh filename="file://$(find arm_urdf)/meshes/link2.stl" scale="0.001 0.001 0.001" />
+                <mesh filename="package://custom_arm_description/meshes/link2.stl" scale="0.001 0.001 0.001" />
             </geometry>
         </collision>
@@ -75,5 +75,5 @@
             <origin xyz="0.2642159907521304 -0.12122484215005706 0.03666668402709977" rpy="-1.4329153603464382 -0.0019516759096357078 -1.5567322881815595" />
             <geometry>
-                <mesh filename="file://$(find arm_urdf)/meshes/link3.stl" scale="0.001 0.001 0.001" />
+                <mesh filename="package://custom_arm_description/meshes/link3.stl" scale="0.001 0.001 0.001" />
             </geometry>
         </visual>
@@ -81,5 +81,5 @@
             <origin xyz="0.2642159907521304 -0.12122484215005706 0.03666668402709977" rpy="-1.4329153603464382 -0.0019516759096357078 -1.5567322881815595" />
             <geometry>
-                <mesh filename="file://$(find arm_urdf)/meshes/link3.stl" scale="0.001 0.001 0.001" />
+                <mesh filename="package://custom_arm_description/meshes/link3.stl" scale="0.001 0.001 0.001" />
             </geometry>
         </collision>
@@ -94,5 +94,5 @@
             <origin xyz="0.07932782337477236 0.2469388385744769 0.08263357936889111" rpy="-3.126581793418305 0.35706491786985606 -1.5675011670871788" />
             <geometry>
-                <mesh filename="file://$(find arm_urdf)/meshes/link4.stl" scale="0.001 0.001 0.001" />
+                <mesh filename="package://custom_arm_description/meshes/link4.stl" scale="0.001 0.001 0.001" />
             </geometry>
         </visual>
@@ -100,5 +100,5 @@
             <origin xyz="0.07932782337477236 0.2469388385744769 0.08263357936889111" rpy="-3.126581793418305 0.35706491786985606 -1.5675011670871788" />
             <geometry>
-                <mesh filename="file://$(find arm_urdf)/meshes/link4.stl" scale="0.001 0.001 0.001" />
+                <mesh filename="package://custom_arm_description/meshes/link4.stl" scale="0.001 0.001 0.001" />
             </geometry>
         </collision>
@@ -113,5 +113,5 @@
             <origin xyz="-0.07070859554835131 -0.23812142491223257 -0.14360878712422676" rpy="1.5861851414203965 -0.013859047172337942 -0.35710948600343884" />
             <geometry>
-                <mesh filename="file://$(find arm_urdf)/meshes/link5.stl" scale="0.001 0.001 0.001" />
+                <mesh filename="package://custom_arm_description/meshes/link5.stl" scale="0.001 0.001 0.001" />
             </geometry>
         </visual>
@@ -119,5 +119,5 @@
             <origin xyz="-0.07070859554835131 -0.23812142491223257 -0.14360878712422676" rpy="1.5861851414203965 -0.013859047172337942 -0.35710948600343884" />
             <geometry>
-                <mesh filename="file://$(find arm_urdf)/meshes/link5.stl" scale="0.001 0.001 0.001" />
+                <mesh filename="package://custom_arm_description/meshes/link5.stl" scale="0.001 0.001 0.001" />
             </geometry>
         </collision>
@@ -132,5 +132,5 @@
             <origin xyz="1.2091060597185789e-09 4.764207801599696e-09 -1.2197904908362035e-10" rpy="-1.5608734092050633 0.2661279038047181 -0.015754050819791802" />
             <geometry>
-                <mesh filename="file://$(find arm_urdf)/meshes/link6.stl" scale="0.001 0.001 0.001" />
+                <mesh filename="package://custom_arm_description/meshes/link6.stl" scale="0.001 0.001 0.001" />
             </geometry>
         </visual>
@@ -138,5 +138,5 @@
             <origin xyz="1.2091060597185789e-09 4.764207801599696e-09 -1.2197904908362035e-10" rpy="-1.5608734092050633 0.2661279038047181 -0.015754050819791802" />
             <geometry>
-                <mesh filename="file://$(find arm_urdf)/meshes/link6.stl" scale="0.001 0.001 0.001" />
+                <mesh filename="package://custom_arm_description/meshes/link6.stl" scale="0.001 0.001 0.001" />
             </geometry>
         </collision>
@@ -151,5 +151,5 @@
             <origin xyz="-0.0022059695912784606 -0.004882435066304681 0.014876005276538429" rpy="3.0578763804063023 -0.2531050091908627 0.3768056949612244" />
             <geometry>
-                <mesh filename="file://$(find arm_urdf)/meshes/Soft_finger_1.stl" scale="0.001 0.001 0.001" />
+                <mesh filename="package://custom_arm_description/meshes/Soft_finger_1.stl" scale="0.001 0.001 0.001" />
             </geometry>
         </visual>
@@ -157,5 +157,5 @@
             <origin xyz="-0.0022059695912784606 -0.004882435066304681 0.014876005276538429" rpy="3.0578763804063023 -0.2531050091908627 0.3768056949612244" />
             <geometry>
-                <mesh filename="file://$(find arm_urdf)/meshes/Soft_finger_1.stl" scale="0.001 0.001 0.001" />
+                <mesh filename="package://custom_arm_description/meshes/Soft_finger_1.stl" scale="0.001 0.001 0.001" />
             </geometry>
         </collision>
@@ -170,5 +170,5 @@
             <origin xyz="-0.003850123319460117 -0.005209890021992578 0.01442336545659309" rpy="-3.1316697359999566 -0.26612790380472257 0.015754050819791247" />
             <geometry>
-                <mesh filename="file://$(find arm_urdf)/meshes/Soft_finger_2.stl" scale="0.001 0.001 0.001" />
+                <mesh filename="package://custom_arm_description/meshes/Soft_finger_2.stl" scale="0.001 0.001 0.001" />
             </geometry>
         </visual>
@@ -176,5 +176,5 @@
             <origin xyz="-0.003850123319460117 -0.005209890021992578 0.01442336545659309" rpy="-3.1316697359999566 -0.26612790380472257 0.015754050819791247" />
             <geometry>
-                <mesh filename="file://$(find arm_urdf)/meshes/Soft_finger_2.stl" scale="0.001 0.001 0.001" />
+                <mesh filename="package://custom_arm_description/meshes/Soft_finger_2.stl" scale="0.001 0.001 0.001" />
             </geometry>
         </collision>
@@ -189,5 +189,5 @@
             <origin xyz="0.0031248681318762194 0.010734304113808584 -0.012592557664950875" rpy="0.8241440367976023 -1.5500870621606404 -2.6609928529842324" />
             <geometry>
-                <mesh filename="file://$(find arm_urdf)/meshes/AX_12A_01.stl" scale="0.001 0.001 0.001" />
+                <mesh filename="package://custom_arm_description/meshes/AX_12A_01.stl" scale="0.001 0.001 0.001" />
             </geometry>
         </visual>
@@ -195,5 +195,5 @@
             <origin xyz="0.0031248681318762194 0.010734304113808584 -0.012592557664950875" rpy="0.8241440367976023 -1.5500870621606404 -2.6609928529842324" />
             <geometry>
-                <mesh filename="file://$(find arm_urdf)/meshes/AX_12A_01.stl" scale="0.001 0.001 0.001" />
+                <mesh filename="package://custom_arm_description/meshes/AX_12A_01.stl" scale="0.001 0.001 0.001" />
             </geometry>
         </collision>
@@ -208,5 +208,5 @@
             <origin xyz="0.0008956910236866023 -0.0025363287034182846 0.012962054304978637" rpy="-2.3174486167921926 1.5500870621606395 2.660992852984249" />
             <geometry>
-                <mesh filename="file://$(find arm_urdf)/meshes/AX_12A_02.stl" scale="0.001 0.001 0.001" />
+                <mesh filename="package://custom_arm_description/meshes/AX_12A_02.stl" scale="0.001 0.001 0.001" />
             </geometry>
         </visual>
@@ -214,5 +214,5 @@
             <origin xyz="0.0008956910236866023 -0.0025363287034182846 0.012962054304978637" rpy="-2.3174486167921926 1.5500870621606395 2.660992852984249" />
             <geometry>
-                <mesh filename="file://$(find arm_urdf)/meshes/AX_12A_02.stl" scale="0.001 0.001 0.001" />
+                <mesh filename="package://custom_arm_description/meshes/AX_12A_02.stl" scale="0.001 0.001 0.001" />
             </geometry>
         </collision>
@@ -227,5 +227,5 @@
             <origin xyz="0.0013596762204496926 0.01195466381035061 0.0023952562436191016" rpy="2.8754522571900396 0.00957358508084527 -1.5891601611840465" />
             <geometry>
-                <mesh filename="file://$(find arm_urdf)/meshes/AX_12A_03.stl" scale="0.001 0.001 0.001" />
+                <mesh filename="package://custom_arm_description/meshes/AX_12A_03.stl" scale="0.001 0.001 0.001" />
             </geometry>
         </visual>
@@ -233,5 +233,5 @@
             <origin xyz="0.0013596762204496926 0.01195466381035061 0.0023952562436191016" rpy="2.8754522571900396 0.00957358508084527 -1.5891601611840465" />
             <geometry>
-                <mesh filename="file://$(find arm_urdf)/meshes/AX_12A_03.stl" scale="0.001 0.001 0.001" />
+                <mesh filename="package://custom_arm_description/meshes/AX_12A_03.stl" scale="0.001 0.001 0.001" />
             </geometry>
         </collision>
@@ -246,5 +246,5 @@
             <origin xyz="0.0017607307048155363 -0.006463816564347109 -9.423452190461036e-05" rpy="-2.317448616792229 1.5500870621606417 2.66099285298433" />
             <geometry>
-                <mesh filename="file://$(find arm_urdf)/meshes/AX_12A_04.stl" scale="0.001 0.001 0.001" />
+                <mesh filename="package://custom_arm_description/meshes/AX_12A_04.stl" scale="0.001 0.001 0.001" />
             </geometry>
         </visual>
@@ -252,5 +252,5 @@
             <origin xyz="0.0017607307048155363 -0.006463816564347109 -9.423452190461036e-05" rpy="-2.317448616792229 1.5500870621606417 2.66099285298433" />
             <geometry>
-                <mesh filename="file://$(find arm_urdf)/meshes/AX_12A_04.stl" scale="0.001 0.001 0.001" />
+                <mesh filename="package://custom_arm_description/meshes/AX_12A_04.stl" scale="0.001 0.001 0.001" />
             </geometry>
         </collision>
@@ -265,5 +265,5 @@
             <origin xyz="0.0010511849185925826 -0.0038589977903183835 -5.625289857050575e-05" rpy="1.5567298120389736 -0.015199409263172443 -2.8754332590191867" />
             <geometry>
-                <mesh filename="file://$(find arm_urdf)/meshes/Gear_Flange_Motor.stl" scale="0.001 0.001 0.001" />
+                <mesh filename="package://custom_arm_description/meshes/Gear_Flange_Motor.stl" scale="0.001 0.001 0.001" />
             </geometry>
         </visual>
@@ -271,5 +271,5 @@
             <origin xyz="0.0010511849185925826 -0.0038589977903183835 -5.625289857050575e-05" rpy="1.5567298120389736 -0.015199409263172443 -2.8754332590191867" />
             <geometry>
-                <mesh filename="file://$(find arm_urdf)/meshes/Gear_Flange_Motor.stl" scale="0.001 0.001 0.001" />
+                <mesh filename="package://custom_arm_description/meshes/Gear_Flange_Motor.stl" scale="0.001 0.001 0.001" />
             </geometry>
         </collision>
@@ -284,5 +284,5 @@
             <origin xyz="0.0023918310966156045 -1.067519965474162e-05 -0.0034947799580093888" rpy="0.08371627318348981 0.2531050091908637 -2.7647869586285765" />
             <geometry>
-                <mesh filename="file://$(find arm_urdf)/meshes/Gear_Flange_Driven.stl" scale="0.001 0.001 0.001" />
+                <mesh filename="package://custom_arm_description/meshes/Gear_Flange_Driven.stl" scale="0.001 0.001 0.001" />
             </geometry>
         </visual>
@@ -290,5 +290,5 @@
             <origin xyz="0.0023918310966156045 -1.067519965474162e-05 -0.0034947799580093888" rpy="0.08371627318348981 0.2531050091908637 -2.7647869586285765" />
             <geometry>
-                <mesh filename="file://$(find arm_urdf)/meshes/Gear_Flange_Driven.stl" scale="0.001 0.001 0.001" />
+                <mesh filename="package://custom_arm_description/meshes/Gear_Flange_Driven.stl" scale="0.001 0.001 0.001" />
             </geometry>
         </collision>

File: final_task/src/custom_arm_description/urdf/gazebo.xacro (robot description, xacro)
@@ -3,15 +3,7 @@
   <!-- ROS 2 Humble / Ignition Gazebo -->
   <gazebo>
-    <xacro:if value="$(arg is_ignition)">
       <plugin filename="ign_ros2_control-system" name="ign_ros2_control::IgnitionROS2ControlPlugin">
-        <parameters>$(find custom_arm_controller)/config/arm_controllers.yaml</parameters>
+        <parameters>$(find custom_arm_moveit)/config/ros2_controllers.yaml</parameters>
       </plugin>
-    </xacro:if>
-    <!-- ROS 2 Iron or above / Gazebo Sim -->
-    <xacro:unless value="$(arg is_ignition)">
-      <plugin filename="gz_ros2_control-system" name="gz_ros2_control::GazeboSimROS2ControlPlugin">
-        <parameters>$(find custom_arm_controller)/config/arm_controllers.yaml</parameters>
-      </plugin>
-    </xacro:unless>
   </gazebo>
 </robot>

File: final_task/src/custom_arm_description/urdf/ros2control.xacro (robot description, xacro)
@@ -3,15 +3,7 @@
   <ros2_control name="RobotSystem" type="system">
     <!-- ROS 2 Humble / Ignition Gazebo -->
-    <xacro:if value="$(arg is_ignition)">
-      <hardware>
-        <plugin>ign_ros2_control/IgnitionSystem</plugin>
-      </hardware>
-    </xacro:if>
-    <!-- ROS 2 Iron or above / Gazebo Sim -->
-    <xacro:unless value="$(arg is_ignition)">
-      <hardware>
-        <plugin>gz_ros2_control/GazeboSimSystem</plugin>
-      </hardware>
-    </xacro:unless>
+    <hardware>
+      <plugin>ign_ros2_control/IgnitionSystem</plugin>
+    </hardware>
     <!-- Joint 1 - Base rotation (z-axis) -->
     <joint name="base_link_link1_to_base_link">
@@ -21,4 +13,5 @@
       </command_interface>
       <state_interface name="position"/>
+      <state_interface name="velocity"/>
     </joint>
     <!-- Joint 2 -->
@@ -29,4 +22,5 @@
       </command_interface>
       <state_interface name="position"/>
+      <state_interface name="velocity"/>
     </joint>
     <!-- Joint 3 -->
@@ -37,4 +31,5 @@
       </command_interface>
       <state_interface name="position"/>
+      <state_interface name="velocity"/>
     </joint>
     <!-- Joint 4 -->
@@ -45,4 +40,5 @@
       </command_interface>
       <state_interface name="position"/>
+      <state_interface name="velocity"/>
     </joint>
     <!-- Joint 5 -->
@@ -53,4 +49,5 @@
       </command_interface>
       <state_interface name="position"/>
+      <state_interface name="velocity"/>
     </joint>
     <!-- Joint 6 -->
@@ -61,4 +58,5 @@
       </command_interface>
       <state_interface name="position"/>
+      <state_interface name="velocity"/>
     </joint>
     <!-- Gripper Joint - Driven Gear -->
@@ -69,4 +67,5 @@
       </command_interface>
       <state_interface name="position"/>
+      <state_interface name="velocity"/>
     </joint>
     <!-- Gripper Joint - Motor Gear -->
@@ -77,4 +76,5 @@
       </command_interface>
       <state_interface name="position"/>
+      <state_interface name="velocity"/>
     </joint>
   </ros2_control>

File: j_ws/src/arm_urdf_moveit_config/config/ArmPlate.ros2_control.xacro (robot description, xacro)
@@ -5,6 +5,5 @@
         <ros2_control name="${prefix}${name}" type="system">
             <hardware>
-                <!-- By default, set up controllers for simulation. This won't work on real hardware -->
-                <plugin>mock_components/GenericSystem</plugin>
+                <plugin>ign_ros2_control/IgnitionSystem</plugin>
             </hardware>
             <joint name="${prefix}Base_link1-v1_Revolute-1">

File: j_ws/src/arm_urdf_moveit_config/config/ArmPlate.xacro (robot description, xacro)
@@ -238,4 +238,12 @@
         <mimic joint="${prefix}gripperHousing-v2_Slider-13" />
     </joint>
+    <gazebo>
+        <plugin filename="ign_ros2_control-system" name="ign_ros2_control::IgnitionROS2ControlPlugin">
+            <parameters>$(find arm_urdf_moveit_config)/config/ros2_controllers.yaml</parameters>
+        </plugin>
+        <plugin filename="ignition-gazebo-sensors-system" name="ignition::gazebo::systems::Sensors">
+            <render_engine>ogre2</render_engine>
+        </plugin>
+    </gazebo>
     </xacro:macro>
 </robot>
