Commit message: Added gripper servo

File: real_shit/src/robot_description/urdf/Arm_assembly.urdf.xacro (robot description, xacro)
@@ -447,4 +447,5 @@
       effort="100"
       velocity="10" />
+    <mimic joint="Jaw" multiplier="-1.0" offset="0.0"/>
   </joint>
   <link

File: real_shit/src/robot_description/urdf/ros2control.xacro (robot description, xacro)
@@ -10,7 +10,7 @@
       <ros2_control name="ArmServoSystem" type="system">
         <hardware>
-          <plugin>arm_servo_controller/ArmServoHardware</plugin>
-          <param name="port">/dev/ttyACM0</param>
-        </hardware>
+	  <plugin>arm_servo_controller/ArmServoHardware</plugin>
+	  <param name="port">/dev/ttyACM0</param>
+	</hardware>
         <joint name="Joint4">
           <command_interface name="position">
@@ -29,4 +29,13 @@
           <param name="id">2</param>
         </joint>
+          <joint name="Jaw">
+            <command_interface name="position">
+              <param name="min">0</param>
+              <param name="max">0.1</param>
+            </command_interface>
+            <state_interface name="position"/>
+            <param name="id">4</param>
+            <param name="type">mg995</param>
+          </joint>
       </ros2_control>
       <ros2_control name="MockArmSystem" type="system">
@@ -52,18 +61,4 @@
             <param name="min">0.0</param>
             <param name="max">2.618</param>
-          </command_interface>
-          <state_interface name="position"/>
-        </joint>
-        <joint name="Jaw">
-          <command_interface name="position">
-            <param name="min">0.0</param>
-            <param name="max">0.1</param>
-          </command_interface>
-          <state_interface name="position"/>
-        </joint>
-        <joint name="Jaw2">
-          <command_interface name="position">
-            <param name="min">-0.1</param>
-            <param name="max">0.0</param>
           </command_interface>
           <state_interface name="position"/>
